File: ASD2501.sch (EAGLE design)
At the start: 23 parts, among them J1 DF12-32-DP, J2 DF12-32-DS, U1 XC6210B18, U2 JF2, U3 TXS0102, U4 TXS0102, Y1 ANT

Commit message: Updated antenna ref des
Parts:
- removed U$2: 0.5pF, tinycircuits:AS-ITM-00126
- removed U$3: 1nH, tinycircuits:AS-ITM-00127
- removed Y1: ANT, akrosense:ANT
- added ANT1: AS-ITM-00109, tinycircuits:AS-ITM-00109
- added C6: 0.5pF, tinycircuits:AS-ITM-00126
- added L1: 1nH, tinycircuits:AS-ITM-00127
Connections:
- net GND: now also ANT1.G1, ANT1.G2, C6.2, L1.2; no longer U$2.2, U$3.2, Y1.G1, Y1.G2
- net N$1: now also C6.1; no longer U$3.1
- net N$5: now also ANT1.1, L1.1; no longer U$2.1, Y1.1
Other:
- moved on the sheet: R5, R9
Changed lines of the file:
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@@
 <setting verticaltext="up"/>
 </settings>
-<grid distance="0.1" unitdist="inch" unit="inch" style="lines" multiple="1" display="no" altdistance="0.01" altunitdist="inch" altunit="inch"/>
+<grid distance="0.01" unitdist="inch" unit="inch" style="lines" multiple="1" display="no" altdistance="0.01" altunitdist="inch" altunit="inch"/>
 <layers>
 <layer number="1" name="Top" color="4" fill="1" visible="no" active="no"/>
@@
 <part name="GND8" library="tinycircuits" deviceset="GND" device=""/>
 <part name="GND9" library="tinycircuits" deviceset="GND" device=""/>
-<part name="Y1" library="akrosense" deviceset="ANT" device=""/>
+<part name="ANT1" library="tinycircuits" deviceset="AS-ITM-00109" device=""/>
 <part name="R2" library="tinycircuits" deviceset="AS-ITM-00076" device="0402_SHORT" value="0.0"/>
 <part name="R3" library="tinycircuits" deviceset="AS-ITM-00076" device="0402_SHORT" value="0.0"/>
@@
 <part name="R5" library="tinycircuits" deviceset="AS-ITM-00076" device="" value="0.0"/>
 <part name="R9" library="tinycircuits" deviceset="AS-ITM-00076" device="" value="0.0"/>
-<part name="U$2" library="tinycircuits" deviceset="AS-ITM-00126" device="" value="0.5pF"/>
-<part name="U$3" library="tinycircuits" deviceset="AS-ITM-00127" device="" value="1nH"/>
+<part name="L1" library="tinycircuits" deviceset="AS-ITM-00127" device="" value="1nH">
+<attribute name="VALUE" value="1nH"/>
+</part>
+<part name="C6" library="tinycircuits" deviceset="AS-ITM-00126" device="" value="0.5pF">
+<attribute name="VALUE" value="0.5pF"/>
+</part>
 </parts>
 <sheets>
@@
 <instance part="GND8" gate="1" x="78.74" y="215.9"/>
 <instance part="GND9" gate="1" x="66.04" y="215.9"/>
-<instance part="Y1" gate="G$1" x="27.94" y="157.48" smashed="yes">
-<attribute name="VALUE" x="29.464" y="150.114" size="1.778" layer="96"/>
+<instance part="ANT1" gate="G$1" x="27.94" y="157.48" smashed="yes">
 <attribute name="NAME" x="20.32" y="160.528" size="1.778" layer="95"/>
 </instance>
@@
 <instance part="GND12" gate="1" x="45.72" y="111.76"/>
 <instance part="GND14" gate="1" x="63.5" y="111.76"/>
-<instance part="R5" gate="G$1" x="53.34" y="134.62"/>
-<instance part="R9" gate="G$1" x="76.2" y="134.62"/>
-<instance part="U$2" gate="G$1" x="45.72" y="124.46"/>
-<instance part="U$3" gate="G$1" x="63.5" y="124.46"/>
+<instance part="R5" gate="G$1" x="55.88" y="134.62"/>
+<instance part="R9" gate="G$1" x="73.66" y="134.62"/>
+<instance part="L1" gate="G$1" x="45.72" y="124.46" smashed="yes">
+<attribute name="NAME" x="48.26" y="124.46" size="1.778" layer="95"/>
+<attribute name="VALUE" x="48.26" y="122.174" size="1.778" layer="96"/>
+</instance>
+<instance part="C6" gate="G$1" x="63.5" y="124.46" smashed="yes">
+<attribute name="NAME" x="67.056" y="124.079" size="1.778" layer="95"/>
+<attribute name="VALUE" x="67.056" y="121.539" size="1.778" layer="96"/>
+</instance>
 </instances>
 <busses>
@@
 </segment>
 <segment>
-<pinref part="Y1" gate="G$1" pin="G2"/>
+<pinref part="ANT1" gate="G$1" pin="G2"/>
 <wire x1="38.1" y1="154.94" x2="40.64" y2="154.94" width="0.1524" layer="91"/>
 <wire x1="40.64" y1="154.94" x2="40.64" y2="152.4" width="0.1524" layer="91"/>
-<pinref part="Y1" gate="G$1" pin="G1"/>
+<pinref part="ANT1" gate="G$1" pin="G1"/>
 <wire x1="38.1" y1="157.48" x2="40.64" y2="157.48" width="0.1524" layer="91"/>
 <wire x1="40.64" y1="157.48" x2="40.64" y2="154.94" width="0.1524" layer="91"/>
@@
 <segment>
 <pinref part="GND12" gate="1" pin="GND"/>
-<pinref part="U$2" gate="G$1" pin="2"/>
-<wire x1="45.72" y1="119.38" x2="45.72" y2="114.3" width="0.1524" layer="91"/>
+<pinref part="L1" gate="G$1" pin="2"/>
+<wire x1="45.72" y1="116.84" x2="45.72" y2="114.3" width="0.1524" layer="91"/>
 </segment>
 <segment>
 <pinref part="GND14" gate="1" pin="GND"/>
-<wire x1="63.5" y1="116.84" x2="63.5" y2="114.3" width="0.1524" layer="91"/>
-<pinref part="U$3" gate="G$1" pin="2"/>
+<wire x1="63.5" y1="119.38" x2="63.5" y2="114.3" width="0.1524" layer="91"/>
+<pinref part="C6" gate="G$1" pin="2"/>
 </segment>
 </net>
@@
 <net name="N$5" class="0">
 <segment>
-<pinref part="Y1" gate="G$1" pin="1"/>
+<pinref part="ANT1" gate="G$1" pin="1"/>
 <wire x1="27.94" y1="147.32" x2="27.94" y2="134.62" width="0.1524" layer="91"/>
-<wire x1="48.26" y1="134.62" x2="45.72" y2="134.62" width="0.1524" layer="91"/>
+<wire x1="50.8" y1="134.62" x2="45.72" y2="134.62" width="0.1524" layer="91"/>
 <wire x1="45.72" y1="134.62" x2="27.94" y2="134.62" width="0.1524" layer="91"/>
 <junction x="45.72" y="134.62"/>
 <pinref part="R5" gate="G$1" pin="1"/>
-<pinref part="U$2" gate="G$1" pin="1"/>
-<wire x1="45.72" y1="127" x2="45.72" y2="134.62" width="0.1524" layer="91"/>
+<pinref part="L1" gate="G$1" pin="1"/>
+<wire x1="45.72" y1="132.08" x2="45.72" y2="134.62" width="0.1524" layer="91"/>
 </segment>
 </net>
@@
 <net name="N$1" class="0">
 <segment>
-<wire x1="58.42" y1="134.62" x2="63.5" y2="134.62" width="0.1524" layer="91"/>
-<wire x1="63.5" y1="134.62" x2="71.12" y2="134.62" width="0.1524" layer="91"/>
-<wire x1="63.5" y1="132.08" x2="63.5" y2="134.62" width="0.1524" layer="91"/>
+<wire x1="60.96" y1="134.62" x2="63.5" y2="134.62" width="0.1524" layer="91"/>
+<wire x1="63.5" y1="134.62" x2="68.58" y2="134.62" width="0.1524" layer="91"/>
+<wire x1="63.5" y1="127" x2="63.5" y2="134.62" width="0.1524" layer="91"/>
 <junction x="63.5" y="134.62"/>
 <pinref part="R5" gate="G$1" pin="2"/>
 <pinref part="R9" gate="G$1" pin="1"/>
-<pinref part="U$3" gate="G$1" pin="1"/>
+<pinref part="C6" gate="G$1" pin="1"/>
 </segment>
 </net>
@@
 <segment>
 <pinref part="U2" gate="G$1" pin="RF_IN"/>
-<wire x1="78.74" y1="134.62" x2="81.28" y2="134.62" width="0.1524" layer="91"/>
 <pinref part="R9" gate="G$1" pin="2"/>
-<wire x1="81.28" y1="134.62" x2="91.44" y2="134.62" width="0.1524" layer="91"/>
-<junction x="81.28" y="134.62"/>
-</segment>
-</net>
+<wire x1="78.74" y1="134.62" x2="91.44" y2="134.62" width="0.1524" layer="91"/>
+</segment>
+</net>
