File: design_files/ASD2501.sch (EAGLE design)
At the start: 23 parts, among them J1 DF12-32-DP, J2 DF12-32-DS, U1 XC6210B18, U2 JF2, U3 TXS0102, U4 TXS0102

Commit message: update format
Parts:
- removed ANT1: AS-ITM-00109, tinycircuits:AS-ITM-00109
- removed L1: 1nH, tinycircuits:AS-ITM-00127
- removed R8: 10.0K, tinycircuits:AS-ITM-00032
- removed R9: 0.0, tinycircuits:AS-ITM-00076
- removed U3, U4: TXS0102, tinycircuits:AS-ITM-00073
- added J3: U.FL-R-SMT(10), tinycircuits:AS-ITM-00193
- added U5: TXB0104, tinycircuits:AS-ITM-00048
- C1, C4: value 0.1uF -> 10uF; device tinycircuits:AS-ITM-00008 -> tinycircuits:AS-ITM-00045; PARTNO AS-ITM-00008 -> AS-ITM-00045; VALUE 0.1uF -> 10uF
- C2: value 47uF -> 0.1uF; device tinycircuits:AS-ITM-00049 -> tinycircuits:AS-ITM-00008; PARTNO (none) -> AS-ITM-00008; PARTNUM AS-ITM-00049 -> (none); VALUE 47uF -> 0.1uF
- C5: value 47uF -> 0.1uF; device tinycircuits:AS-ITM-00049 -> tinycircuits:AS-ITM-00008; PARTNO (none) -> AS-ITM-00008; VALUE (none) -> 0.1uF
- C6: value 0.5pF -> 100pF; device tinycircuits:AS-ITM-00126 -> tinycircuits:AS-ITM-00148; PARTNO (none) -> AS-ITM-00148; VALUE 0.5pF -> 100pF
- R2, R3: device tinycircuits:AS-ITM-000760402_SHORT -> tinycircuits:AS-ITM-00076; VALUE (none) -> 0.0
- R5: PARTNO (none) -> AS-ITM-00076; VALUE (none) -> 0.0
Connections:
- removed net N$5 (its old number): ANT1.1, L1.1, R5.1
- new net N$14: U2.GPIO7
- new net N$6: R7.2, U1.NC/GO
- net AD2: now also R5.2; no longer R7.2
- net AD3: now also U5.B2; no longer U4.B1
- net GND: now also J3.GND1, J3.GND2, R7.1, U2.NC4, U5.GND; no longer ANT1.G1, ANT1.G2, C6.2, L1.2, U3.GND, U4.GND
- net N$1: now also J3.ANT; no longer R5.2, R9.1
- net N$10: no longer R8.2
- net N$11: now also U5.A2; no longer U4.A1
- net N$12: now also U5.A1; no longer U4.A2
- net N$13: now also R5.1, U5.B1; no longer R7.1, U4.B2
- net N$2: now also U5.B3; no longer U3.B1
- net N$3: now also U5.B4; no longer U3.B2
- net N$4: now also U5.A3; no longer U3.A1
- net N$7: now also U5.A4; no longer U3.A2
- net N$8: now also C5.1; no longer C4.1
- net N$9: now also C6.2; no longer R9.2
- net VCC: now also U5.VCCB; no longer U3.VCCB, U4.VCCB
- net VCC_1V8: now also C4.1, U5.OE, U5.VCCA; no longer C5.1, R8.1, U3.OE, U3.VCCA, U4.OE, U4.VCCA
Other:
- note added: "4"
- note added: "Hand Populated: J3, U2"
- note added: "Hand Soldered: -"
- note added: "Non Populated: R1, R4, R7"
- note added: "Notes:"
- note added: "Telit SE868 V2/JF2 GPS Module"
- note added: "Variant: Standard - R"
- note removed: "3"
- note removed: "Telit JF2 GPS Module"
- moved on the sheet: C1, C2, C3, C4, C5, C6, R1, R2, R3, R4, R5, R6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
